File: Custom ESP Controller/CustmESPController/CustmESPController.kicad_sch (KiCad schematic)
At the start: 143 parts, among them IC1 SMD_IC_SY8089AAAC, IC2 ESP32-C6-WROOM-1-N4, IC3 MAX3232EIDR, J1 Screw_Terminal_01x02, J10 J1B1211CCD, J11 DE9_Plug, J12 DE9_Plug, J13 Screw_Terminal_01x02, J14 Screw_Terminal_01x02, J15 Conn_01x03_Pin, J16 Conn_01x03_Pin, J17 USB_C_Receptacle_USB2.0_16P, J18 Screw_Terminal_01x02, J19 Screw_Terminal_01x02, J2 Screw_Terminal_01x03, J20 Screw_Terminal_01x02, J21 Screw_Terminal_01x02, J22 Conn_01x05_Pin, J3 Screw_Terminal_01x02, J4 Conn_01x03_Pin, J5 Conn_01x03_Pin, J6 Conn_01x03_Pin, J7 Conn_01x03_Pin, J8 Conn_01x03_Pin, J9 Conn_01x03_Pin, Q1 WPM2015-3/TR, Q2 SS8050-G(RANGE:120-200), Q3 SS8050-G(RANGE:120-200), Q4 IRLML6244, Q5 IRLML6244, Q6 IRLML6244, Q7 IRLML6244, SW1 SW_Push, SW2 SW_Push, T1 LMUN2235LT1G(SOT-23), T2 LMUN2235LT1G(SOT-23), U2 W5500, U3 CP2102N-Axx-xQFN28, Y1 Crystal_GND24

Commit message: 3D PCB done
Parts:
- removed D7: 1N4148W(SOD-123), OLIMEX_Diodes-FP:SOD-123_1C-2A_KA, symbol ESP32-C6-EVB_Rev_A:D
- removed J13: Screw_Terminal_01x02, symbol Connector:Screw_Terminal_01x02
- removed J2: Screw_Terminal_01x03, symbol Connector:Screw_Terminal_01x03
- removed LED1, LED2: LED/GREEN/0603, OLIMEX_LEDs-FP:LED_0603_KA, symbol ESP32-C6-EVB_Rev_A:LED
- removed R35, R36: 2.2k/R0402, OLIMEX_RLC-FP:R_0402_5MIL_DWS, symbol ESP32-C6-EVB_Rev_A:R
- removed REL1, REL2: RAS-0515, OLIMEX_Relays-FP:Relay_RAS-05-15, symbol ESP32-C6-EVB_Rev_A:Relay
- removed SW1, SW2: SW_Push, symbol Switch:SW_Push
- removed T2: LMUN2235LT1G(SOT-23), OLIMEX_Transistors-FP:SOT23, symbol ESP32-C6-EVB_Rev_A:LMUN2235LT1G(SOT-23)
- added D11: 1N4148W(SOD-123), customESP_Controller:1N4148W_SODFL3816X120N, symbol ESP32-C6-EVB_Rev_A:D
- added H1, H2, H3, H4: ~, MountingHole:MountingHole_2.2mm_M2, symbol Mechanical:MountingHole
- added J2: Screw_Terminal_01x02, TerminalBlock:TerminalBlock_Altech_AK300-2_P5.00mm, symbol Connector:Screw_Terminal_01x02
- added J23: 694106301002, customESP_Controller:694106301002_1, symbol ESP_Project:694106301002
- added K1, K2: SRD-05VDC-SL-C, customESP_Controller:RELAY_SRD-05VDC-SL-C, symbol CustomESP:SRD-05VDC-SL-C
- added SW1, SW2: TS665CJ, Button_Switch_THT:SW_PUSH_6mm, symbol Switch:SW_Push_Dual
- added T3: LMUN2235LT1G(SOT-23), customESP_Controller:LMUN2235LT1G, symbol ESP32-C6-EVB_Rev_A:LMUN2235LT1G(SOT-23)
- C1, C10, C11, C19, C2, C20, C3, C37, C38, C39, C40, C41, C7, C8: footprint (none) -> Capacitor_SMD:C_0603_1608Metric
- C12, C13, C14, C15, C16, C17, C18, C21, C22, C23, C24, C25, C26, C27, C28, C29, C30, C4, C9: footprint (none) -> Capacitor_SMD:C_0402_1005Metric
- C5: value C_Polarized -> 470uF/10V/RVT1A471M0607; footprint (none) -> Capacitor_SMD:CP_Elec_6.3x7.7
- C6: value 100uF/63V/20%/10x13MM/Low_ESR/RM5 -> 100uF/63V/LV101M063G105ETR; footprint (none) -> Capacitor_SMD:CP_Elec_10x10.5
- D1: footprint (none) -> LED_SMD:LED_0603_1608Metric
- D10, D2, D9: value D_TVS -> LESD5D5.0CT1G; footprint (none) -> customESP_Controller:LESD5D5.0CT1G_DTVS
- D3: footprint OLIMEX_Diodes-FP:SOD-123_1C-2A_KA -> customESP_Controller:1N4148W_SODFL3816X120N
- D4: footprint Diode_SMD:D_SMA -> customESP_Controller:SMAJ58A_DIOM5026X229N
- D5: footprint Diode_SMD:D_SMA -> customESP_Controller:DIO_SS310
- D6: footprint Diode_THT:D_DO-201AD_P15.24mm_Horizontal -> customESP_Controller:1N5822_DIOAD3070W130L950D530
- D8: footprint lib:LED_D5.0mm-4_RGB -> LED_THT:LED_D5.0mm-4_RGB
- IC1: footprint SOT95P285X140-5N -> customESP_Controller:SY80B9AAAC_SOT95P285X140-5N
- IC2: footprint ESP32C6WROOM1N4 -> customESP_Controller:ESP32C6WROOM1N4
- IC3: footprint SOIC127P600X175-16N -> customESP_Controller:MAX3232EIDR_SOIC127P600X175-16N
- J1, J14, J18, J19, J20, J21, J3: footprint (none) -> TerminalBlock:TerminalBlock_Altech_AK300-2_P5.00mm
- J10: footprint J1B1211CCD -> customESP_Controller:J1B1211CCD
- J11, J12: footprint (none) -> Connector_Dsub:DSUB-9_Female_Vertical_P2.77x2.84mm_MountingHoles
- J15, J16: footprint (none) -> Connector_JST:JST_EH_B3B-EH-A_1x03_P2.50mm_Vertical
- J17: footprint lib:HRO_TYPE-C-31-M-12 -> Connector_USB:USB_C_Receptacle_HRO_TYPE-C-31-M-12
- J22: footprint (none) -> Connector_JST:JST_EH_B5B-EH-A_1x05_P2.50mm_Vertical
- J4, J5, J6, J7, J8, J9: footprint (none) -> Connector_PinHeader_2.54mm:PinHeader_1x03_P2.54mm_Vertical
- L1: value 33uH/2.1A/DCR=0.1R/20%/DBS135(PD3316MT330) -> 33uH/SL0630-330M; footprint (none) -> customESP_Controller:SL0630-330M
- L2: footprint (none) -> customESP_Controller:IND_NR3015T2R2M
- L3: footprint (none) -> Inductor_SMD:L_0603_1608Metric
- Q1: footprint (none) -> customESP_Controller:WPM2015-3TR_SOT95P240X130-3N
- Q2, Q3: footprint lib:SS8050-G -> customESP_Controller:SS8050_SOT95P240X115-3N
- Q4, Q5, Q6, Q7: value IRLML6244 -> IRLML6244TRPBF; footprint Package_TO_SOT_SMD:SOT-23 -> customESP_Controller:IRLML6244TRPBF_SOT95P237X112-3N
- R1, R10, R11, R12, R13, R14, R15, R16, R17, R18, R19, R2, R20, R21, R23, R24, R25, R26, R27, R28, R29, R3, R30, R31, R4, R48, R49, R7, R8, R9: footprint (none) -> Resistor_SMD:R_0402_1005Metric
- R22: footprint (none) -> Resistor_SMD:R_1206_3216Metric
- R46, R47, R5, R6: value R -> 100R; footprint (none) -> Resistor_SMD:R_0402_1005Metric
- T1: footprint OLIMEX_Transistors-FP:SOT23 -> customESP_Controller:LMUN2235LT1G
- TX4138(ESOIC-8)1: renamed from TX1; footprint (none) -> customESP_Controller:TX4138_SOIC127P600X165-9N
- U2: footprint Package_QFP:LQFP-48_7x7mm_P0.5mm -> customESP_Controller:W5500_QFP50P900X900X160-48N
- U3: footprint Package_DFN_QFN:QFN-28-1EP_5x5mm_P0.5mm_EP3.35x3.35mm -> customESP_Controller:CP2102N_QFN50P500X500X80-29N-D
- Y1: value Crystal_GND24 -> HSO321S 24MHZ 3.3V -40~+85℃; footprint (none) -> customESP_Controller:HSO321S
Connections:
- net +12V: now also J23.1 (POWER)
- net +5V: now also D11.1 (K), K1.A1, K2.A1
- net ESP_EN: now also SW1.1
- net GND: now also J11.0 (GND), J12.0 (GND), J23.2 (GND_1), J23.3 (GND_2), SW1.2, SW2.2, T3.2 (E); no longer C23.1, C24.1, R10.2, R11.1, U2.30 (XI/CLKIN), Y1.1, Y1.3
- net GPIO11/REL2: now also T3.1 (B)
- net at D3.2 (A): now also K2.A2, T3.3 (C); no longer T1.3 (C)
- net at J14.1 (Pin_1): now also K1.NO
- net at J14.2 (Pin_2): now also K1.COM
- net at R8.2: now also SW2.1
- new net: J2.1 (Pin_1), K2.NO
- new net: J2.2 (Pin_2), K2.COM
- new net: C24.1, R10.2, Y1.3
- new net: D11.2 (A), K1.A2, T1.3 (C)
- new net XI: C23.1, R11.1, U2.30 (XI/CLKIN), Y1.1
Other:
- note added: "DC Barrel"
- moved on the sheet: C24, J14, J19, J20, T1
